Commit message: wedgebot

File: sumogym/robot_descriptions/simple_robot/simple_robot_2.urdf (robot description, URDF)
Before this commit: robot differential_drive_robot, 4 links, 3 joints
Links:
- removed link caster
- link base_link: geometry collision mesh filename=body.stl; visual mesh filename=body.stl
- link left_wheel: mass 1 -> 0.2; geometry collision cylinder length=0.05 radius=0.14; visual cylinder length=0.05 radius=0.14
- link right_wheel: mass 1 -> 0.2; geometry collision cylinder length=0.05 radius=0.14; visual cylinder length=0.05 radius=0.14
Joints:
- removed joint base_link_to_caster
- joint left_wheel_joint: origin xyz=0 0.15 0 -> xyz=0.02 0.175 0 rpy=0 0 0
- joint right_wheel_joint: origin xyz=0 -0.15 0 -> xyz=0.02 -0.175 0 rpy=0 0 0

Commit message: single control working

File: sumogym/robot_descriptions/simple_robot/simple_robot_2.urdf (robot description, URDF)
Before this commit: robot differential_drive_robot, 3 links, 2 joints
Links:
- link base_link: mass 5 -> 2.3
